Commit message: Update box.urdf

File: envs/assets/bulletobjects/box/box2/box.urdf (robot description, URDF)
Before this commit: robot bowl.urdf, 2 links, 1 joints
Links:
- added link base2, mass .1; collision box size=.05 1 .5; collision box size=.05 1 .5
- link base: geometry collision box size=1 1 .1; visual box size=1 1 .1
Joints:
- added joint base_joint2: type fixed, parent base, child base2
