Commit message: Update rectangularprism2.urdf

File: envs/assets/bulletobjects/obj/rectangularprism2.urdf (robot description, URDF)
Before this commit: robot cube.urdf, 1 links, 0 joints
Links:
- link cube: mass 0.01 -> 0.05

Commit message: Update rectangularprism2.urdf

File: envs/assets/bulletobjects/obj/rectangularprism2.urdf (robot description, URDF)
Before this commit: robot cube.urdf, 1 links, 0 joints
Links:
- removed link cube
- added link rectangularprism2, mass 0.03; collision box size=1 1 1.75; visual box size=1 1 1.75
