Commit message: Update tetris1.urdf

File: envs/assets/bulletobjects/obj/tetris1.urdf (robot description, URDF)
Before this commit: robot tetris1.urdf, 3 links, 2 joints
Links:
- link center: geometry collision box size=1.8 1 1; visual box size=1.8 1 1
Joints:
- joint fixed1: origin xyz=1 0 0 rpy=0 0 0 -> xyz=1.1 0 0 rpy=0 0 0
- joint fixed2: origin xyz=-1 0 0 rpy=0 0 0 -> xyz=-1.1 0 0 rpy=0 0 0
